File: electrical/pi-zero-board/open-race-scale-pi-zero-board-v.01.sch (EAGLE design)
At the start: 64 parts, among them J5 PIN20X2, Q1 MMBT4403, Q2 MMBT4403, Q3 MMBT4403, Q4 MMBT4403, U1 HX711, U2 HX711, U3 HX711, U4 HX711

Commit message: first rev of pi zero integrated board
is compatible with all RPi, zero is used to control costs
Connections:
- net B+2 renamed N$14
- net B-2 renamed N$15
- removed net B+1: JP5.1, JP7.1, U3.INB+, U4.INB+
- removed net B-1: JP5.2, JP7.2, U3.INB-, U4.INB-
- new net N$11: JP5.1, U3.INB+
- new net N$12: JP5.2, U3.INB-
- new net N$13: JP7.2, U4.INB-
- new net N$8: JP7.1, U4.INB+
