File: electrical/pi-zero-board/open-race-scale-pi-zero-board-v.02.brd (EAGLE design)
At the start: 78.7 x 40.3 mm, 64 parts, among them J5 PIN20X2, Q1 MMBT4403, Q2 MMBT4403, Q3 MMBT4403, Q4 MMBT4403, U1 HX711, U2 HX711, U3 HX711, U4 HX711

Commit message: board passes etc and drc
Parts:
- added H1, H2, H3, H4: MOUNT-HOLE3.3, holes:3,3
- JP1, JP2, JP5, JP7: device SparkFun-Connectors:1X02 -> SparkFun-Connectors:1X02@1
- SJ1, SJ2, SJ3, SJ4: device SparkFun-Passives:PAD-JUMPER-2-NC_BY_TRACE_YES_SILK -> SparkFun-Connectors:1X02
- moved SJ2 21.7 mm to (59.7, 57.1), turned to 90 degrees
- moved SJ1 20.5 mm to (40.6, 57.1), turned to 90 degrees
- moved R5 20.3 mm to (59.7, 67.3)
- moved R10 19.0 mm to (40.6, 67.3), turned to 90 degrees
- moved SJ3 7.73 mm to (21.6, 57.1), turned to 90 degrees
- moved SJ4 7.73 mm to (78.7, 57.1), turned to 90 degrees
- moved C9 2.54 mm to (29.2, 74.9)
- moved R20 1.80 mm to (78.7, 66.0), turned to 90 degrees
- moved R15 1.27 mm to (19.1, 68.6), turned to 180 degrees
- moved C21 1.27 mm to (45.7, 76.2)
- turned C3 to 90 degrees
- turned C7 to 90 degrees
Routing:
- net N$122: track 38.0 -> 14.1 mm, vias 0 -> 2
- net N$1: track 23.5 -> 12.2 mm, vias 0 -> 2
- net N$191: track 4.37 -> 15.5 mm, vias 0 -> 2
- net GND: track 340.0 -> 332.4 mm, vias 2 -> 16
- net N$26: track 3.48 -> 10.6 mm
- net AVDD2: track 61.5 -> 64.4 mm
- net VCC: track 217.7 -> 220.5 mm, vias 6 -> 7
- net VDD: track 128.7 -> 131.1 mm
- net SCK2: track 25.1 -> 26.4 mm
Other:
- board size 78.7 x 40.3 mm -> 96.5 x 45.4 mm
