File: electrical/pi-zero-board/open-race-scale-pi-zero-board-v.02.sch (EAGLE design)
At the start: 64 parts, among them J5 PIN20X2, Q1 MMBT4403, Q2 MMBT4403, Q3 MMBT4403, Q4 MMBT4403, U1 HX711, U2 HX711, U3 HX711, U4 HX711

Commit message: board passes etc and drc
Parts:
- added H1, H2, H3, H4: MOUNT-HOLE3.3, holes:MOUNT-HOLE3.3
- SJ1, SJ2, SJ3, SJ4: value JUMPER-PAD-2-NC_BY_TRACE -> (none); device SparkFun-Passives:JUMPER-PAD-2-NC_BY_TRACE -> SparkFun-Connectors:CONN_02
Changed lines of the file:
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@@
 <part name="C2" library="SparkFun-Capacitors" deviceset="0.1UF-25V-5%(0603)" device="" value="0.1uF"/>
 <part name="JP2" library="SparkFun-Connectors" deviceset="M02" device="PTH"/>
-<part name="SJ2" library="SparkFun-Passives" deviceset="JUMPER-PAD-2-NC_BY_TRACE" device="" value=""/>
+<part name="SJ2" library="SparkFun-Connectors" deviceset="CONN_02" device=""/>
 <part name="JP4" library="SparkFun-Connectors" deviceset="M05" device="PTH"/>
 <part name="C3" library="SparkFun-Capacitors" deviceset="0.1UF-25V-5%(0603)" device="" value="0.1uF"/>
@@
 <part name="C12" library="SparkFun-Capacitors" deviceset="0.1UF-25V-5%(0603)" device="" value="0.1uF"/>
 <part name="JP1" library="SparkFun-Connectors" deviceset="M02" device="PTH"/>
-<part name="SJ1" library="SparkFun-Passives" deviceset="JUMPER-PAD-2-NC_BY_TRACE" device="" value=""/>
+<part name="SJ1" library="SparkFun-Connectors" deviceset="CONN_02" device=""/>
 <part name="JP3" library="SparkFun-Connectors" deviceset="M05" device="PTH"/>
 <part name="C13" library="SparkFun-Capacitors" deviceset="0.1UF-25V-5%(0603)" device="" value="0.1uF"/>
@@
 <part name="GND27" library="SparkFun-Aesthetics" deviceset="GND" device=""/>
 <part name="JP5" library="SparkFun-Connectors" deviceset="M02" device="PTH"/>
-<part name="SJ3" library="SparkFun-Passives" deviceset="JUMPER-PAD-2-NC_BY_TRACE" device="" value=""/>
+<part name="SJ3" library="SparkFun-Connectors" deviceset="CONN_02" device=""/>
 <part name="JP6" library="SparkFun-Connectors" deviceset="M05" device="PTH"/>
 <part name="C20" library="SparkFun-Capacitors" deviceset="0.1UF-25V-5%(0603)" device="" value="0.1uF"/>
@@
 <part name="C26" library="SparkFun-Capacitors" deviceset="0.1UF-25V-5%(0603)" device="" value="0.1uF"/>
 <part name="JP7" library="SparkFun-Connectors" deviceset="M02" device="PTH"/>
-<part name="SJ4" library="SparkFun-Passives" deviceset="JUMPER-PAD-2-NC_BY_TRACE" device="" value=""/>
+<part name="SJ4" library="SparkFun-Connectors" deviceset="CONN_02" device=""/>
 <part name="JP8" library="SparkFun-Connectors" deviceset="M05" device="PTH"/>
 <part name="C27" library="SparkFun-Capacitors" deviceset="0.1UF-25V-5%(0603)" device="" value="0.1uF"/>
@@
 <part name="L4" library="SparkFun-Passives" deviceset="INDUCTOR" device="0805-IND" value="3.3uH"/>
 <part name="J5" library="FLYFISH" deviceset="PIN20X2" device=""/>
+<part name="H1" library="holes" deviceset="MOUNT-HOLE" device="3.3"/>
+<part name="H2" library="holes" deviceset="MOUNT-HOLE" device="3.3"/>
+<part name="H3" library="holes" deviceset="MOUNT-HOLE" device="3.3"/>
+<part name="H4" library="holes" deviceset="MOUNT-HOLE" device="3.3"/>
 </parts>
 <sheets>
@@
 <instance part="C2" gate="G$1" x="58.42" y="43.18" rot="R90"/>
 <instance part="JP2" gate="G$1" x="-22.86" y="48.26"/>
-<instance part="SJ2" gate="G$1" x="111.76" y="68.58" rot="R90"/>
+<instance part="SJ2" gate="G$1" x="121.92" y="68.58" rot="MR0"/>
 <instance part="JP4" gate="G$1" x="-22.86" y="68.58"/>
 <instance part="C3" gate="G$1" x="7.62" y="66.04"/>
@@
 <instance part="C12" gate="G$1" x="50.8" y="170.18" rot="R90"/>
 <instance part="JP1" gate="G$1" x="-30.48" y="175.26"/>
-<instance part="SJ1" gate="G$1" x="104.14" y="195.58" rot="R90"/>
+<instance part="SJ1" gate="G$1" x="111.76" y="195.58" rot="MR0"/>
 <instance part="JP3" gate="G$1" x="-30.48" y="195.58"/>
 <instance part="C13" gate="G$1" x="0" y="193.04"/>
@@
 <instance part="GND27" gate="1" x="10.16" y="317.5"/>
 <instance part="JP5" gate="G$1" x="-35.56" y="279.4"/>
-<instance part="SJ3" gate="G$1" x="99.06" y="299.72" rot="R90"/>
+<instance part="SJ3" gate="G$1" x="106.68" y="299.72" rot="MR0"/>
 <instance part="JP6" gate="G$1" x="-35.56" y="299.72"/>
 <instance part="C20" gate="G$1" x="-5.08" y="297.18"/>
@@
 <instance part="C26" gate="G$1" x="66.04" y="-83.82" rot="R90"/>
 <instance part="JP7" gate="G$1" x="-15.24" y="-78.74"/>
-<instance part="SJ4" gate="G$1" x="119.38" y="-58.42" rot="R90"/>
+<instance part="SJ4" gate="G$1" x="134.62" y="-60.96" rot="MR0"/>
 <instance part="JP8" gate="G$1" x="-15.24" y="-58.42"/>
 <instance part="C27" gate="G$1" x="15.24" y="-60.96"/>
@@
 </instance>
 <instance part="J5" gate="G$1" x="223.52" y="119.38" rot="R180"/>
+<instance part="H1" gate="G$1" x="7.62" y="114.3"/>
+<instance part="H2" gate="G$1" x="7.62" y="109.22"/>
+<instance part="H3" gate="G$1" x="7.62" y="104.14"/>
+<instance part="H4" gate="G$1" x="7.62" y="99.06"/>
 </instances>
 <busses>
@@
 <segment>
 <pinref part="GND7" gate="1" pin="GND"/>
-<wire x1="111.76" y1="63.5" x2="111.76" y2="60.96" width="0.1524" layer="91"/>
 <pinref part="SJ2" gate="G$1" pin="1"/>
+<wire x1="114.3" y1="68.58" x2="111.76" y2="60.96" width="0.1524" layer="91"/>
 </segment>
 <segment>
@@
 <segment>
 <pinref part="GND16" gate="1" pin="GND"/>
-<wire x1="104.14" y1="190.5" x2="104.14" y2="187.96" width="0.1524" layer="91"/>
+<wire x1="104.14" y1="195.58" x2="104.14" y2="187.96" width="0.1524" layer="91"/>
 <pinref part="SJ1" gate="G$1" pin="1"/>
 </segment>
@@
 <segment>
 <pinref part="GND26" gate="1" pin="GND"/>
-<wire x1="99.06" y1="294.64" x2="99.06" y2="292.1" width="0.1524" layer="91"/>
+<wire x1="99.06" y1="299.72" x2="99.06" y2="292.1" width="0.1524" layer="91"/>
 <pinref part="SJ3" gate="G$1" pin="1"/>
 </segment>
@@
 <segment>
 <pinref part="GND36" gate="1" pin="GND"/>
-<wire x1="119.38" y1="-63.5" x2="119.38" y2="-66.04" width="0.1524" layer="91"/>
+<wire x1="127" y1="-60.96" x2="119.38" y2="-66.04" width="0.1524" layer="91"/>
 <pinref part="SJ4" gate="G$1" pin="1"/>
 </segment>
@@
 <wire x1="99.06" y1="68.58" x2="104.14" y2="68.58" width="0.1524" layer="91"/>
 <wire x1="111.76" y1="78.74" x2="111.76" y2="76.2" width="0.1524" layer="91"/>
-<wire x1="111.76" y1="76.2" x2="111.76" y2="73.66" width="0.1524" layer="91"/>
+<wire x1="111.76" y1="76.2" x2="114.3" y2="71.12" width="0.1524" layer="91"/>
 <wire x1="111.76" y1="76.2" x2="104.14" y2="76.2" width="0.1524" layer="91"/>
 <wire x1="104.14" y1="76.2" x2="104.14" y2="68.58" width="0.1524" layer="91"/>
@@
 <wire x1="91.44" y1="195.58" x2="96.52" y2="195.58" width="0.1524" layer="91"/>
 <wire x1="104.14" y1="205.74" x2="104.14" y2="203.2" width="0.1524" layer="91"/>
-<wire x1="104.14" y1="203.2" x2="104.14" y2="200.66" width="0.1524" layer="91"/>
+<wire x1="104.14" y1="203.2" x2="104.14" y2="198.12" width="0.1524" layer="91"/>
 <wire x1="104.14" y1="203.2" x2="96.52" y2="203.2" width="0.1524" layer="91"/>
 <wire x1="96.52" y1="203.2" x2="96.52" y2="195.58" width="0.1524" layer="91"/>
@@
 <wire x1="86.36" y1="299.72" x2="91.44" y2="299.72" width="0.1524" layer="91"/>
 <wire x1="99.06" y1="309.88" x2="99.06" y2="307.34" width="0.1524" layer="91"/>
-<wire x1="99.06" y1="307.34" x2="99.06" y2="304.8" width="0.1524" layer="91"/>
+<wire x1="99.06" y1="307.34" x2="99.06" y2="302.26" width="0.1524" layer="91"/>
 <wire x1="99.06" y1="307.34" x2="91.44" y2="307.34" width="0.1524" layer="91"/>
 <wire x1="91.44" y1="307.34" x2="91.44" y2="299.72" width="0.1524" layer="91"/>
@@
 <wire x1="106.68" y1="-58.42" x2="111.76" y2="-58.42" width="0.1524" layer="91"/>
 <wire x1="119.38" y1="-48.26" x2="119.38" y2="-50.8" width="0.1524" layer="91"/>
-<wire x1="119.38" y1="-50.8" x2="119.38" y2="-53.34" width="0.1524" layer="91"/>
+<wire x1="119.38" y1="-50.8" x2="127" y2="-58.42" width="0.1524" layer="91"/>
 <wire x1="119.38" y1="-50.8" x2="111.76" y2="-50.8" width="0.1524" layer="91"/>
 <wire x1="111.76" y1="-50.8" x2="111.76" y2="-58.42" width="0.1524" layer="91"/>
@@
 </sheet>
 </sheets>
+<errors>
+</errors>
 </schematic>
 </drawing>
