File: electrical/pi-zero-board/open-race-scale-pi-zero-board-v.03.sch (EAGLE design)
At the start: 68 parts, among them J5 PIN20X2, Q1 MMBT4403, Q2 MMBT4403, Q3 MMBT4403, Q4 MMBT4403, U1 HX711, U2 HX711, U3 HX711, U4 HX711

Commit message: silk screen
Connections:
- net N$11 renamed B+1
- net N$12 renamed B-1
- net N$13 renamed B-4
- net N$14 renamed B+2
- net N$15 renamed B-2
- net N$8 renamed B+4
Changed lines of the file:
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@@
 </segment>
 </net>
-<net name="N$8" class="0">
+<net name="B+4" class="0">
 <segment>
 <pinref part="U4" gate="U1" pin="INB+"/>
@@
 <pinref part="JP7" gate="G$1" pin="1"/>
 <wire x1="-7.62" y1="-119.38" x2="-7.62" y2="-78.74" width="0.1524" layer="91"/>
+<label x="-2.54" y="-81.28" size="1.778" layer="95" rot="R180"/>
 </segment>
 </net>
-<net name="N$11" class="0">
+<net name="B+1" class="0">
 <segment>
 <pinref part="U3" gate="U1" pin="INB+"/>
@@
 <pinref part="JP5" gate="G$1" pin="1"/>
 <wire x1="-27.94" y1="236.22" x2="-27.94" y2="279.4" width="0.1524" layer="91"/>
+<label x="-27.94" y="274.32" size="1.778" layer="95" rot="R180"/>
 </segment>
 </net>
-<net name="N$12" class="0">
+<net name="B-1" class="0">
 <segment>
 <pinref part="JP5" gate="G$1" pin="2"/>
@@
 <pinref part="U3" gate="U1" pin="INB-"/>
 <wire x1="86.36" y1="243.84" x2="86.36" y2="269.24" width="0.1524" layer="91"/>
+<label x="-22.86" y="281.94" size="1.778" layer="95"/>
 </segment>
 </net>
-<net name="N$13" class="0">
+<net name="B-4" class="0">
 <segment>
 <pinref part="JP7" gate="G$1" pin="2"/>
@@
 <pinref part="U4" gate="U1" pin="INB-"/>
 <wire x1="106.68" y1="-111.76" x2="106.68" y2="-88.9" width="0.1524" layer="91"/>
+<label x="0" y="-73.66" size="1.778" layer="95" rot="R180"/>
 </segment>
 </net>
-<net name="N$14" class="0">
+<net name="B+2" class="0">
 <segment>
 <pinref part="JP1" gate="G$1" pin="1"/>
@@
 <pinref part="U2" gate="U1" pin="INB+"/>
 <wire x1="104.14" y1="170.18" x2="91.44" y2="170.18" width="0.1524" layer="91"/>
+<label x="-17.78" y="175.26" size="1.778" layer="95" rot="R180"/>
 </segment>
 </net>
-<net name="N$15" class="0">
+<net name="B-2" class="0">
 <segment>
 <pinref part="JP1" gate="G$1" pin="2"/>
@@
 <pinref part="U2" gate="U1" pin="INB-"/>
 <wire x1="91.44" y1="139.7" x2="91.44" y2="165.1" width="0.1524" layer="91"/>
+<label x="-15.24" y="180.34" size="1.778" layer="95" rot="R180"/>
 </segment>
 </net>
